File: Electronic Design/Etch_sAo_Sketch_V0.1 Design Files KiCAD 8/Etch_sAo_Sketch.kicad_pcb (KiCad board)
At the start: 2 copper layers, 50.8 x 76.8 mm, 38 parts, among them Q22 SL3401A, U1 LIS2DH, U2 SC18IS606PWJ, U7 SSP9193-33M5R, X1 SAO_conn_SFH11-NBPC-D03-ST-BK, X2 SAO_conn_SFH11-NBPC-D03-ST-BK, X3 HEADER_4-PIN_0.1, X4 HEADER_11-PIN_0.1, X5 HEADER_11-PIN_0.1

Commit message: Remove top SAO port
Parts:
- removed JP21: V_SEL, Jumper:SolderJumper-3_P1.3mm_Bridged12_Pad1.0x1.5mm
- removed X2: SAO_conn_SFH11-NBPC-D03-ST-BK, Andy_Footprint_Library:Badgelife-SAOv169-BADGE-2x3-no-front-text
- removed X4: HEADER_11-PIN_0.1, Connector_PinSocket_2.54mm:PinSocket_1x11_P2.54mm_Vertical
- moved L2 17.8 mm to (74.5, 170.3)
- moved kibuzzard-6417AF30 15.3 mm to (113.9, 96.6)
Routing:
- net GND: track 150.0 -> 2.87 mm
- net /GPIO1: track 119.5 -> 0.00 mm
- net /GPIO2: track 115.4 -> 0.00 mm
- net /SDA: track 111.2 -> 0.00 mm
- net VIN: track 107.5 -> 0.00 mm
- net unconnected-(RV1-Pad1): track 106.1 -> 0.00 mm
- net 3V3: track 84.9 -> 0.00 mm
- net Net-(Q22-S): track 42.7 -> 0.00 mm
- net /3V3_LDO: track 6.90 -> 0.00 mm
- net Net-(U7-BP): track 2.37 -> 0.00 mm
- net Net-(Q22-G): track 2.26 -> 0.00 mm
Other:
- board size 50.8 x 76.8 mm -> 50.8 x 70.4 mm
