File: Electronic Design/Etch_sAo_Sketch_V0.1 Design Files KiCAD 8/Etch_sAo_Sketch.kicad_sch (KiCad schematic)
At the start: 36 parts, among them Q22 SL3401A, U1 LIS2DH, U2 SC18IS606PWJ, U7 SSP9193-33M5R, X1 SAO_conn_SFH11-NBPC-D03-ST-BK, X2 SAO_conn_SFH11-NBPC-D03-ST-BK, X3 HEADER_4-PIN_0.1, X4 HEADER_11-PIN_0.1, X5 HEADER_11-PIN_0.1

Commit message: Remove top SAO port
Parts:
- removed JP21: V_SEL, Jumper:SolderJumper-3_P1.3mm_Bridged12_Pad1.0x1.5mm, symbol Jumper:SolderJumper_3_Bridged12
- removed X2: SAO_conn_SFH11-NBPC-D03-ST-BK, Andy_Footprint_Library:Badgelife-SAOv169-BADGE-2x3-no-front-text, symbol ANDY_SYMBOL_LIBRARY:SAO_conn_SFH11-NBPC-D03-ST-BK-badgelife_shitty_addon_v169bis
- removed X4: HEADER_11-PIN_0.1, Connector_PinSocket_2.54mm:PinSocket_1x11_P2.54mm_Vertical, symbol Connector_Generic:Conn_01x11
Connections:
- no-connect marks 2 -> 1
Other:
- note added: "ACCELEROMETER"
- note added: "ANALOG KNOBS"
- note added: "EPAPER"
- note added: "I2C TO SPI BRIDGE"
- note removed: "Compatible: https://www.adafruit.com/product/1431 1.5” 128x128, 16-bit color w/MicroSD holder OLED has 5V -> 3V3 regulator onboard. MicroSD card standalone pins shared between TFT and OLED boards."
- note removed: "GPIO EXPANDER"
- note removed: "OLED COLOR SPI W/MICRO SD"
- note removed: "SAO #2 (OUT/TOP)"
- moved on the sheet: U1, U2
