File: Electronic Design/Etch_sAo_Sketch_V1.0 Design Files KiCAD 8/Etch_sAo_Sketch.kicad_sch (KiCad schematic)
At the start: 16 parts, among them U2 LIS3DHTR, X1 SAO_conn_SFH11-NBPC-D03-ST-BK, X3 OLED_128x128

Commit message: Add schematic for V1 OLED
Other:
- note added: "LIS3DHTR 3-AXIS Accel 0x19 with SDO/SA0 high (default) LIS3DHTR 3-AXIS Accel 0x18 with SDO/SA0 low (remove R1 and jumper pin 7 to ground) OLED 128x128 1.5 inch SSD1327 0x3C (dec 60)"
- note removed: "LIS3DHTR 3-AXIS Accel 0x19 with SA0 high. OLED 128x128 1.5 inch SSD1327 0x3C (dec 60)"
Changed lines of the file:
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@@
 		)
 	)
-	(text "LIS3DHTR 3-AXIS Accel               0x19 with SA0 high.\nOLED 128x128 1.5 inch SSD1327     0x3C (dec 60)"
+	(text "LIS3DHTR 3-AXIS Accel               0x19 with SDO/SA0 high (default)\nLIS3DHTR 3-AXIS Accel               0x18 with SDO/SA0 low (remove R1 and jumper pin 7 to ground)\nOLED 128x128 1.5 inch SSD1327     0x3C (dec 60)"
 		(exclude_from_sim no)
-		(at 99.822 171.831 0)
+		(at 16.256 185.547 0)
 		(effects
 			(font
@@
 	(text "I2C ADDRESS TABLE"
 		(exclude_from_sim no)
-		(at 99.06 159.385 0)
+		(at 15.494 173.101 0)
 		(effects
 			(font
@@
 	(text "All 7-bit addresses should be greater\nthan 0x07 and less than 0x78 (120)."
 		(exclude_from_sim no)
-		(at 100.33 163.83 0)
+		(at 16.764 177.546 0)
 		(effects
 			(font
