File: Electronic Design/SAO_Sketch_V1.3 Design Files KiCAD 8/SAO_Sketch.kicad_sch (KiCad schematic)
At the start: 17 parts, among them U1 LIS3DHTR, X1 SAO_conn_SFH11-NBPC-D03-ST-BK, X2 OLED_128x128

Commit message: Add I2C pull-up errata notes and SAO_Sketch_V1.3 Schematic Errata 2025-04-01.pdf
Too much combined I2C pull-up resistance!
Other:
- note added: "ERRATA 2025-04-01"
- note added: "SAO SKETCH - OLED VERSION (V1.3) FOR HACKADAY EUROPE 2025"
- note added: "There is too much combined pull-up resistance with this board, the OLED board, the Hackaday Badge, and the Pico. This inhibits I2C hardware implementations from working with the OLED display. SOLUTION A: Firmware workaround is to use software I2C. See: https://github.com/ageppert/SAO_Etch_sAo_Sketch/pull/1 SOLUTION B: Hardware mods to remove interfering components. See: https://github.com/agepper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"
- note removed: "SAO SKETCH - OLED VERSION FOR HACKADAY EUROPE 2025"
Changed lines of the file:
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@@
 		)
 	)
-	(text "SAO SKETCH - OLED VERSION\nFOR HACKADAY EUROPE 2025"
+	(text "SAO SKETCH - OLED VERSION\n(V1.3) FOR HACKADAY EUROPE 2025"
 		(exclude_from_sim no)
 		(at 140.208 31.75 0)
@@
 		)
 	)
+	(text "There is too much combined pull-up resistance with this board,\nthe OLED board, the Hackaday Badge, and the Pico. This inhibits\nI2C hardware implementations from working with the OLED display.\nSOLUTION A: Firmware workaround is to use software I2C.\n   See: https://github.com/ageppert/SAO_Etch_sAo_Sketch/pull/1\nSOLUTION B: Hardware mods to remove interfering components.\n   See: https://github.com/ageppert/SAO_Etch_sAo_Sketch/issues/8"
+		(exclude_from_sim no)
+		(at 159.766 165.608 0)
+		(effects
+			(font
+				(size 1.524 1.524)
+				(thickness 1.6)
+				(bold yes)
+				(color 255 0 0 1)
+			)
+			(justify left bottom)
+		)
+	)
 	(text "ACCELEROMETER"
 		(exclude_from_sim no)
@@
 		)
 	)
+	(text "ERRATA 2025-04-01"
+		(exclude_from_sim no)
+		(at 158.496 145.796 0)
+		(effects
+			(font
+				(size 6 6)
+				(thickness 1.6)
+				(bold yes)
+				(color 255 0 0 1)
+			)
+			(justify left bottom)
+		)
+	)
 	(label "SDA"
 		(at 32.385 64.77 0)
-		(fields_autoplaced yes)
 		(effects
 			(font
@@
 	(label "GPIO1"
 		(at 32.385 67.31 0)
-		(fields_autoplaced yes)
 		(effects
 			(font
@@
 	(label "SCL"
 		(at 32.385 87.63 0)
-		(fields_autoplaced yes)
 		(effects
 			(font
@@
 	(label "POT2R"
 		(at 254 66.04 0)
-		(fields_autoplaced yes)
 		(effects
 			(font
@@
 	(label "INT2"
 		(at 201.93 105.41 90)
-		(fields_autoplaced yes)
 		(effects
 			(font
@@
 	(label "GPIO2"
 		(at 32.385 85.09 0)
-		(fields_autoplaced yes)
 		(effects
 			(font
@@
 	(label "GPIO1"
 		(at 185.42 96.52 0)
-		(fields_autoplaced yes)
 		(effects
 			(font
@@
 	(label "SCL"
 		(at 119.38 67.31 0)
-		(fields_autoplaced yes)
 		(effects
 			(font
@@
 	(label "SDA"
 		(at 72.39 64.77 0)
-		(fields_autoplaced yes)
 		(effects
 			(font
@@
 	(label "GPIO2"
 		(at 185.42 111.76 0)
-		(fields_autoplaced yes)
 		(effects
 			(font
@@
 	(label "POT1L"
 		(at 223.52 66.04 0)
-		(fields_autoplaced yes)
 		(effects
 			(font
@@
 	(label "SDA"
 		(at 119.38 64.77 0)
-		(fields_autoplaced yes)
 		(effects
 			(font
@@
 	(label "SCL"
 		(at 72.39 67.31 0)
-		(fields_autoplaced yes)
 		(effects
 			(font
@@
 	(label "INT1"
 		(at 195.58 90.17 90)
-		(fields_autoplaced yes)
-		(effects
-			(font
+		(effects
+			(font
